File: Tempic-HW/Tempic-HW.kicad_pcb (KiCad board)
At the start: 2 copper layers, 50 x 50 mm, 56 parts, among them J1 BMV080, J2 Conn_01x08_Pin, J3 Conn_01x08_Pin, P1 217175-0001, U1 ESP32-C6-MINI-1, U2 BQ25504, U3 BME688, U4 TPS631000, U5 MCP73831-2-MC, U6 TPS62A01PDDC, Y1 32.7680k

Commit message: Finished PCB, added silkscreen graphics.
Parts:
- added ?: , , F.Cu at (117.9, 136.0)
- added C13: 100n, Capacitor_SMD:C_0402_1005Metric_Pad0.74x0.62mm_HandSolder, F.Cu at (132.7, 97.2)
- added D3: ESDZV5-1BV2, Diode_SMD:Nexperia_DSN0603-2_0.6x0.3mm_P0.4mm, F.Cu at (137.3, 130.5)
- added REF**: MountingHole_2.2mm_M2_DIN965_Pad, MountingHole:MountingHole_2.2mm_M2_DIN965_Pad, F.Cu at (162.0, 97.8)
- added REF**: MountingHole_2.2mm_M2_DIN965_Pad, MountingHole:MountingHole_2.2mm_M2_DIN965_Pad, F.Cu at (162.0, 136.0)
- moved SC1 37.2 mm to (117.9, 122.0)
- moved U1 36.9 mm to (125.5, 134.4), turned to 180 degrees
- moved L1 36.0 mm to (125.0, 119.2)
- moved BT1 33.4 mm to (117.9, 129.3)
- moved D1 31.1 mm to (128.2, 134.5), turned to -90 degrees
- moved U4 30.4 mm to (132.9, 116.5), turned to 180 degrees
- moved Y1 29.9 mm to (135.6, 107.6), turned to 180 degrees
- moved P1 28.9 mm to (140.0, 139.0)
- moved C7 25.0 mm to (144.1, 112.3), turned to 180 degrees
- moved R13 24.6 mm to (141.7, 129.8), turned to 90 degrees
- moved R20 23.4 mm to (131.2, 100.3), turned to 180 degrees
- moved C2 22.8 mm to (121.0, 122.6), turned to -90 degrees
- moved R19 22.5 mm to (131.2, 99.3)
- moved U3 21.4 mm to (144.2, 115.6), turned to 90 degrees
- moved C14 20.0 mm to (132.6, 103.0), turned to -90 degrees
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- renumbered C8 to C1, C14 to C10, C7 to C11, C15 to C12, C10 to C14, C18 to C15, C11 to C16, C16 to C18, C12 to C19, C4 to C2, C1 to C3, C3 to C4, C9 to C5, C2 to C6, C13 to C7, C5 to C8, C6 to C9, L2 to L1, L1 to L2, R7 to R1, R5 to R10, R10 to R11, R11 to R12, R20 to R13, R15 to R14, R16 to R15, R17 to R16, R1 to R17, R2 to R18, R18 to R19, R8 to R2, R19 to R20, R13 to R3, R9 to R4, R6 to R5, R14 to R6, R12 to R7, R3 to R8, R4 to R9, U5 to U1, U6 to U3, U1 to U5, U3 to U6
Connections:
- U1 pad 9: (no net) -> GND
Routing:
- net +3.3V: track 0.00 -> 135.1 mm, vias 0 -> 5
- net +2.5V: track 0.00 -> 72.2 mm, vias 0 -> 4
- net +5V: track 0.00 -> 55.4 mm, vias 0 -> 3
- net /SDA: track 0.00 -> 51.3 mm, vias 0 -> 3
- net /BAT: track 0.00 -> 48.9 mm, vias 0 -> 3
- net /STAT: track 0.00 -> 45.1 mm, vias 0 -> 4
- net /IO20: track 0.00 -> 40.7 mm, vias 0 -> 1
- net /IO23: track 0.00 -> 40.7 mm, vias 0 -> 1
- net /IO22: track 0.00 -> 40.1 mm, vias 0 -> 1
- net /IO21: track 0.00 -> 40.1 mm, vias 0 -> 1
- net /SCL: track 0.00 -> 39.9 mm, vias 0 -> 3
- net Net-(U2-VSTOR): track 0.00 -> 32.8 mm, vias 0 -> 2
- net /IO18: track 0.00 -> 31.2 mm, vias 0 -> 1
- net /USB_D+: track 0.00 -> 30.0 mm, vias 0 -> 2
- net /USB_D-: track 0.00 -> 29.7 mm
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- added copper zone on B.Cu, net GND
- added copper zone on F.Cu, net GND
Other:
- board size 50 x 50 mm -> 50 x 45.3 mm
- board text added: "18.9.2026"
- board text added: "2.5V"
- board text added: "2.5V BUCK"
- board text added: "3.3V"
- board text added: "3.3V P.S."
- board text added: "5V"
- board text added: "BAT"
- board text added: "BAT CHRG"
- board text added: "BME688"
- board text added: "BMV080"
- board text added: "Developed with love by: Jernej Leskovec"
- board text added: "ESP32 C6"
- board text added: "GND"
- board text added: "IO15"
- board text added: "IO18"
- board text added: "IO19"
- board text added: "IO20"
- board text added: "IO21"
- board text added: "IO22"
- board text added: "IO23"
- board text added: "IO3"
- board text added: "IO4"
- board text added: "IO5"
- board text added: "RXDO"
- board text added: "SLR"
- board text added: "SOLAR"
- board text added: "TXDO"
- board text added: "Tempic 1.0"
- board text added: "USB 2.0"
- board text added: "USB-C"
- board text added: "WiFi 6"
- board text added: "Zigbee 3"

Commit message: Chandeg hysteresis of battery charging and edited README.
Parts:
- BT1: value Battery_Cell -> LiPo
- R10: value 332k -> 316k
- R11: value 5.49M -> 5.62M
- R12: value 4.12M -> 4.02M

Commit message: Fixed PCB edge.
Other:
- outline, holes or cut-outs redrawn
Changed lines of the file:
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@@
 		(layer "F.Cu")
 		(at 140 139.01)
-		(property "Reference" "P1"
-			(at 1.73 -9.145 0)
-			(layer "F.SilkS")
+		(property "Datasheet" ""
+			(at 0 0 0)
+			(layer "F.Fab")
 			(hide yes)
 			(effects
 				(font
-					(size 1 1)
-					(thickness 0.15)
+					(size 1.27 1.27)
 				)
 			)
 		)
-		(property "Value" "217175-0001"
-			(at 0 -10.5575 0)
+		(property "Description" "USB 2.0-only Type-C Plug connector"
+			(at 0 0 0)
 			(layer "F.Fab")
+			(hide yes)
 			(effects
 				(font
-					(size 1 1)
-					(thickness 0.15)
+					(size 1.27 1.27)
 				)
 			)
 		)
-		(property "Datasheet" ""
-			(at 0 0 0)
+		(property "Value" "217175-0001"
+			(at 0 -10.5575 0)
 			(layer "F.Fab")
-			(hide yes)
 			(effects
 				(font
-					(size 1.27 1.27)
+					(size 1 1)
+					(thickness 0.15)
 				)
 			)
 		)
-		(property "Description" "USB 2.0-only Type-C Plug connector"
-			(at 0 0 0)
-			(layer "F.Fab")
+		(property "Reference" "P1"
+			(at 1.73 -9.145 0)
+			(layer "F.SilkS")
 			(hide yes)
 			(effects
 				(font
-					(size 1.27 1.27)
+					(size 1 1)
+					(thickness 0.15)
 				)
 			)
@@
 		(sheetname "/")
 		(sheetfile "Tempic-HW.kicad_sch")
-		(units
-			(unit
-				(name "A")
-				(pins "SH" "A8" "B8" "A1" "A12" "A4" "A9" "A5" "B5" "A7" "B7" "A6" "B6")
-			)
-		)
 		(attr smd)
 		(duplicate_pad_numbers_are_jumpers no)
@@
 		(fp_line
 			(start -3.6 -8.35)
-			(end -2.8 -8.350001)
+			(end -2.8 -8.35)
 			(stroke
 				(width 0.15)
@@
 		)
 		(fp_line
-			(start -2.8 -8.350001)
+			(start -2.8 -8.35)
 			(end -3.2 -9.05)
 			(stroke
@@
 			(layer "Edge.Cuts")
 		)
-		(fp_line
-			(start 4.62 0)
-			(end -4.62 0)
-			(stroke
-				(width 0.01)
-				(type solid)
-			)
-			(layer "Edge.Cuts")
-		)
 		(fp_arc
 			(start -4.62 -6.700001)
 			(mid -4.397644 -6.989779)
-			(end -4.060189 -6.85)
+			(end -4.06019 -6.85)
 			(stroke
 				(width 0.01)
@@
 		)
 		(fp_arc
-			(start 4.060189 -6.85)
-			(mid 3.950381 -6.740192)
+			(start 4.06019 -6.85)
+			(mid 3.95038 -6.740198)
 			(end 3.80038 -6.7)
 			(stroke
@@
 		(fp_arc
 			(start 4.060191 -6.85)
-			(mid 4.397645 -6.989778)
+			(mid 4.397646 -6.989779)
 			(end 4.62 -6.7)
 			(stroke
@@
 		)
 		(fp_line
-			(start -6.420001 0.3)
-			(end 6.420001 0.3)
+			(start -6.42 -8.1)
+			(end -6.42 0.3)
 			(stroke
 				(width 0.01)
@@
 		)
 		(fp_line
-			(start -6.42 -8.099999)
-			(end -6.420001 0.3)
+			(start -6.42 0.3)
+			(end 6.42 0.3)
 			(stroke
 				(width 0.01)
@@
 		)
 		(fp_line
-			(start 6.42 -8.099999)
-			(end -6.42 -8.099999)
+			(start 6.42 -8.1)
+			(end -6.42 -8.1)
 			(stroke
 				(width 0.01)
@@
 		)
 		(fp_line
-			(start 6.420001 0.3)
-			(end 6.42 -8.099999)
+			(start 6.42 0.3)
+			(end 6.42 -8.1)
 			(stroke
 				(width 0.01)
@@
 		)
 		(fp_line
-			(start -4.47 0)
-			(end 4.47 0)
-			(stroke
-				(width 0.13)
-				(type solid)
-			)
-			(layer "F.Fab")
-		)
-		(fp_line
 			(start -3.80038 -6.7)
 			(end 3.80038 -6.7)
@@
 		(fp_line
 			(start -3.6 -8.35)
-			(end -2.8 -8.350001)
+			(end -2.8 -8.35)
 			(stroke
 				(width 0.13)
@@
 		)
 		(fp_line
-			(start -2.8 -8.350001)
+			(start -2.8 -8.35)
 			(end -3.2 -9.05)
 			(stroke
@@
 			(start -4.62 -6.700001)
 			(mid -4.397644 -6.989779)
-			(end -4.060189 -6.85)
+			(end -4.06019 -6.85)
 			(stroke
 				(width 0.13)
@@
 		)
 		(fp_arc
-			(start 4.060189 -6.85)
-			(mid 3.950381 -6.740192)
+			(start 4.06019 -6.85)
+			(mid 3.95038 -6.740198)
 			(end 3.80038 -6.7)
 			(stroke
@@
 		(fp_arc
 			(start 4.060191 -6.85)
-			(mid 4.397645 -6.989778)
+			(mid 4.397646 -6.989779)
 			(end 4.62 -6.7)
 			(stroke
@@
 		)
 		(pad "SH" thru_hole oval
-			(at -5.62 -6.099999)
+			(at -5.62 -6.1)
 			(size 1 1.8)
 			(drill oval 0.6 1.4)
@@
 		)
 		(pad "SH" thru_hole oval
-			(at 5.62 -6.099999)
+			(at 5.62 -6.1)
 			(size 1 1.8)
 			(drill oval 0.6 1.4)
@@
 		(layer "F.SilkS")
 	)
-	(gr_rect
+	(gr_line
+		(start 115 93.7)
+		(end 115 139)
+		(stroke
+			(width 0.05)
+			(type default)
+		)
+		(layer "Edge.Cuts")
+	)
+	(gr_line
 		(start 115 93.7)
+		(end 165 93.7)
+		(stroke
+			(width 0.05)
+			(type default)
+		)
+		(layer "Edge.Cuts")
+	)
+	(gr_line
+		(start 115 139)
+		(end 135.38 139.01)
+		(stroke
+			(width 0.05)
+			(type default)
+		)
+		(layer "Edge.Cuts")
+	)
+	(gr_line
+		(start 165 93.7)
 		(end 165 139)
 		(stroke
@@
 			(type default)
 		)
-		(fill no)
+		(layer "Edge.Cuts")
+	)
+	(gr_line
+		(start 165 139)
+		(end 144.62 139.01)
+		(stroke
+			(width 0.05)
+			(type default)
+		)
 		(layer "Edge.Cuts")
 	)
